File: ee/ovrdrive/ovrdrive.kicad_sch (KiCad schematic)
At the start: 44 parts, among them J1 USB_A, J3 AVR-ISP-6, U1 SM3257ENT, U2 FLASH, U3 ATtiny24A-MM, U4 SN74LVC1G32DCKR, U5 DRV8837C

Commit message: R0.41 released.
Parts:
- C14, C3: value 1uF -> 10uF; MPN (none) -> CL10A106MQ8NNNC
- J3: value AVR-ISP-6 -> TC2030; footprint Connector_PinHeader_1.27mm:PinHeader_2x03_P1.27mm_Horizontal -> Connector:Tag-Connect_TC2030-IDC-NL_2x03_P1.27mm_Vertical; MPN 20021112-00006T4LF -> TC2030; now left out of the parts list
- R5: value 2.2R -> 0R; MPN RC0603FR-072R2L -> RC0603FR-070RL
Other:
- company: (none) -> Interrupt Labs
- title: (none) -> Overdrive
Changed lines of the file:
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@@
 (kicad_sch (version 20230121) (generator eeschema)
   (paper "A4")
+  (title_block
+    (title "Overdrive")
+    (date "2024-01-11")
+    (rev "R0.41")
+    (company "Interrupt Labs")
+    (comment 1 "Ryan Walker")
+    (comment 2 "Walker@interruptlabs.ca")
+  )
   (junction (at 74.93 125.095) (diameter 0) (color 0 0 0 0)
   )
@@
     (stroke (width 0) (type default))
   )
-  (wire (pts (xy 32.385 53.975) (xy 27.94 53.975))
-    (stroke (width 0) (type default))
-  )
   (wire (pts (xy 80.645 125.095) (xy 82.55 125.095))
     (stroke (width 0) (type default))
@@
     (stroke (width 0) (type default))
   )
+  (wire (pts (xy 41.91 51.435) (xy 41.91 53.975))
+    (stroke (width 0) (type default))
+  )
   (wire (pts (xy 73.025 125.095) (xy 74.93 125.095))
     (stroke (width 0) (type default))
@@
     (stroke (width 0) (type default))
   )
+  (wire (pts (xy 27.94 53.975) (xy 32.385 53.975))
+    (stroke (width 0) (type default))
+  )
   (wire (pts (xy 37.465 53.975) (xy 41.91 53.975))
     (stroke (width 0) (type default))
@@
     (stroke (width 0) (type default))
   )
-  (wire (pts (xy 41.91 50.165) (xy 41.91 53.975))
-    (stroke (width 0) (type default))
-  )
   (wire (pts (xy 104.775 85.725) (xy 99.06 85.725))
     (stroke (width 0) (type default))
@@
       (effects (font (size 1.27 1.27)) (justify left))
     )
-    (property "Value" "1uF" (at 24.765 181.61 0)
+    (property "Value" "10uF" (at 24.765 181.61 0)
       (effects (font (size 1.27 1.27)) (justify left))
     )
@@
       (effects (font (size 1.27 1.27)) hide)
     )
-    (property "MPN" "" (at 26.035 183.515 0)
+    (property "MPN" "CL10A106MQ8NNNC" (at 26.035 183.515 0)
       (effects (font (size 1.27 1.27)) hide)
     )
@@
   )
   (symbol (lib_id "Connector:AVR-ISP-6") (at 34.29 142.875 0) (unit 1)
-    (in_bom yes) (on_board yes) (dnp no) (fields_autoplaced)
+    (in_bom no) (on_board yes) (dnp no) (fields_autoplaced)
     (property "Reference" "J3" (at 25.4 140.335 0)
       (effects (font (size 1.27 1.27)) (justify right))
     )
-    (property "Value" "AVR-ISP-6" (at 25.4 142.875 0)
+    (property "Value" "TC2030" (at 25.4 142.875 0)
       (effects (font (size 1.27 1.27)) (justify right))
     )
-    (property "Footprint" "Connector_PinHeader_1.27mm:PinHeader_2x03_P1.27mm_Horizontal" (at 27.94 141.605 90)
+    (property "Footprint" "Connector:Tag-Connect_TC2030-IDC-NL_2x03_P1.27mm_Vertical" (at 27.94 141.605 90)
       (effects (font (size 1.27 1.27)) hide)
     )
@@
       (effects (font (size 1.27 1.27)) hide)
     )
-    (property "MPN" "20021112-00006T4LF" (at 34.29 142.875 0)
+    (property "MPN" "TC2030" (at 34.29 142.875 0)
       (effects (font (size 1.27 1.27)) hide)
     )
@@
       (effects (font (size 1.27 1.27)) (justify left))
     )
-    (property "Value" "1uF" (at 53.34 181.61 0)
+    (property "Value" "10uF" (at 53.34 181.61 0)
       (effects (font (size 1.27 1.27)) (justify left))
     )
@@
       (effects (font (size 1.27 1.27)) hide)
     )
-    (property "MPN" "" (at 54.61 183.515 0)
+    (property "MPN" "CL10A106MQ8NNNC" (at 54.61 183.515 0)
       (effects (font (size 1.27 1.27)) hide)
     )
@@
     )
   )
-  (symbol (lib_id "power:+5V") (at 41.91 50.165 0) (unit 1)
+  (symbol (lib_id "power:+5V") (at 41.91 51.435 0) (unit 1)
     (in_bom yes) (on_board yes) (dnp no) (fields_autoplaced)
-    (property "Reference" "#PWR0102" (at 41.91 53.975 0)
+    (property "Reference" "#PWR0102" (at 41.91 55.245 0)
       (effects (font (size 1.27 1.27)) hide)
     )
-    (property "Value" "+5V" (at 41.91 46.5892 0)
+    (property "Value" "+5V" (at 41.91 47.8592 0)
       (effects (font (size 1.27 1.27)))
     )
-    (property "Footprint" "" (at 41.91 50.165 0)
+    (property "Footprint" "" (at 41.91 51.435 0)
       (effects (font (size 1.27 1.27)) hide)
     )
-    (property "Datasheet" "" (at 41.91 50.165 0)
+    (property "Datasheet" "" (at 41.91 51.435 0)
       (effects (font (size 1.27 1.27)) hide)
     )
@@
       (effects (font (size 1.27 1.27)) (justify left))
     )
-    (property "Value" "2.2R" (at 33.02 52.705 90)
+    (property "Value" "0R" (at 33.02 52.705 90)
       (effects (font (size 1.27 1.27)) (justify left))
     )
@@
       (effects (font (size 1.27 1.27)) hide)
     )
-    (property "MPN" "RC0603FR-072R2L" (at 34.925 53.975 90)
+    (property "MPN" "RC0603FR-070RL" (at 34.925 53.975 90)
       (effects (font (size 1.27 1.27)) hide)
     )
